File: pcb/display.brd (EAGLE design)
At the start: 99 x 95.2 mm, 37 parts, among them IC1 74HC595D, IC2 74HC595D

Commit message: edit pcb
Routing:
- net N$11: track 114.8 -> 110.3 mm
- net N$34: track 67.9 -> 71.5 mm
- net N$27: track 73.8 -> 76.8 mm
Changed lines of the file:
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@@
 <grid distance="0.05" unitdist="inch" unit="inch" style="lines" multiple="1" display="yes" altdistance="0.025" altunitdist="inch" altunit="inch"/>
 <layers>
-<layer number="1" name="Top" color="4" fill="1" visible="no" active="yes"/>
+<layer number="1" name="Top" color="4" fill="1" visible="yes" active="yes"/>
 <layer number="2" name="Route2" color="1" fill="3" visible="no" active="no"/>
 <layer number="3" name="Route3" color="4" fill="3" visible="no" active="no"/>
@@
 <layer number="14" name="Route14" color="1" fill="6" visible="no" active="no"/>
 <layer number="15" name="Route15" color="4" fill="6" visible="no" active="no"/>
-<layer number="16" name="Bottom" color="1" fill="1" visible="no" active="yes"/>
+<layer number="16" name="Bottom" color="1" fill="1" visible="yes" active="yes"/>
 <layer number="17" name="Pads" color="2" fill="1" visible="yes" active="yes"/>
-<layer number="18" name="Vias" color="2" fill="1" visible="no" active="yes"/>
+<layer number="18" name="Vias" color="2" fill="1" visible="yes" active="yes"/>
 <layer number="19" name="Unrouted" color="6" fill="1" visible="yes" active="yes"/>
 <layer number="20" name="Dimension" color="15" fill="1" visible="yes" active="yes"/>
-<layer number="21" name="tPlace" color="7" fill="1" visible="yes" active="yes"/>
-<layer number="22" name="bPlace" color="7" fill="1" visible="yes" active="yes"/>
-<layer number="23" name="tOrigins" color="15" fill="1" visible="yes" active="yes"/>
-<layer number="24" name="bOrigins" color="15" fill="1" visible="yes" active="yes"/>
+<layer number="21" name="tPlace" color="7" fill="1" visible="no" active="yes"/>
+<layer number="22" name="bPlace" color="7" fill="1" visible="no" active="yes"/>
+<layer number="23" name="tOrigins" color="15" fill="1" visible="no" active="yes"/>
+<layer number="24" name="bOrigins" color="15" fill="1" visible="no" active="yes"/>
 <layer number="25" name="tNames" color="7" fill="1" visible="yes" active="yes"/>
 <layer number="26" name="bNames" color="7" fill="1" visible="yes" active="yes"/>
@@
 <wire x1="49.53" y1="74.93" x2="52.07" y2="74.93" width="0.6096" layer="16"/>
 <wire x1="26.67" y1="74.93" x2="24.13" y2="74.93" width="0.6096" layer="16"/>
-<wire x1="22.86" y1="80.01" x2="48.26" y2="80.01" width="0.6096" layer="16"/>
-<wire x1="48.26" y1="80.01" x2="49.53" y2="78.74" width="0.6096" layer="16"/>
-<wire x1="49.53" y1="78.74" x2="49.53" y2="74.93" width="0.6096" layer="16"/>
-<wire x1="74.93" y1="74.93" x2="74.93" y2="78.74" width="0.6096" layer="16"/>
-<wire x1="74.93" y1="78.74" x2="73.66" y2="80.01" width="0.6096" layer="16"/>
-<wire x1="73.66" y1="80.01" x2="50.8" y2="80.01" width="0.6096" layer="16"/>
-<wire x1="50.8" y1="80.01" x2="49.53" y2="78.74" width="0.6096" layer="16"/>
-<wire x1="22.86" y1="80.01" x2="21.59" y2="78.74" width="0.6096" layer="16"/>
+<wire x1="24.13" y1="81.28" x2="48.26" y2="81.28" width="0.6096" layer="16"/>
+<wire x1="48.26" y1="81.28" x2="49.53" y2="80.01" width="0.6096" layer="16"/>
+<wire x1="49.53" y1="80.01" x2="49.53" y2="74.93" width="0.6096" layer="16"/>
+<wire x1="74.93" y1="74.93" x2="74.93" y2="80.01" width="0.6096" layer="16"/>
+<wire x1="74.93" y1="80.01" x2="73.66" y2="81.28" width="0.6096" layer="16"/>
+<wire x1="73.66" y1="81.28" x2="54.61" y2="81.28" width="0.6096" layer="16"/>
+<wire x1="54.61" y1="81.28" x2="53.34" y2="80.01" width="0.6096" layer="16"/>
+<wire x1="53.34" y1="80.01" x2="49.53" y2="80.01" width="0.6096" layer="16"/>
+<wire x1="24.13" y1="81.28" x2="21.59" y2="78.74" width="0.6096" layer="16"/>
 <wire x1="21.59" y1="78.74" x2="21.59" y2="76.2" width="0.6096" layer="16"/>
 <wire x1="21.59" y1="76.2" x2="22.86" y2="74.93" width="0.6096" layer="16"/>
@@
 <wire x1="29.21" y1="73.66" x2="29.21" y2="74.93" width="0.6096" layer="16"/>
 <wire x1="29.21" y1="74.93" x2="29.21" y2="77.47" width="0.6096" layer="16"/>
-<wire x1="29.21" y1="77.47" x2="30.48" y2="78.74" width="0.6096" layer="16"/>
-<wire x1="30.48" y1="78.74" x2="45.72" y2="78.74" width="0.6096" layer="16"/>
-<wire x1="45.72" y1="78.74" x2="46.99" y2="77.47" width="0.6096" layer="16"/>
-<wire x1="46.99" y1="77.47" x2="46.99" y2="74.93" width="0.6096" layer="16"/>
+<wire x1="29.21" y1="77.47" x2="31.75" y2="80.01" width="0.6096" layer="16"/>
+<wire x1="31.75" y1="80.01" x2="45.72" y2="80.01" width="0.6096" layer="16"/>
+<wire x1="45.72" y1="80.01" x2="46.99" y2="78.74" width="0.6096" layer="16"/>
+<wire x1="46.99" y1="78.74" x2="46.99" y2="74.93" width="0.6096" layer="16"/>
 <wire x1="46.99" y1="74.93" x2="46.99" y2="72.39" width="0.6096" layer="16"/>
 <wire x1="46.99" y1="72.39" x2="48.26" y2="71.12" width="0.6096" layer="16"/>
@@
 <wire x1="54.61" y1="72.39" x2="54.61" y2="74.93" width="0.6096" layer="16"/>
 <wire x1="54.61" y1="74.93" x2="54.61" y2="77.47" width="0.6096" layer="16"/>
-<wire x1="54.61" y1="77.47" x2="55.88" y2="78.74" width="0.6096" layer="16"/>
-<wire x1="55.88" y1="78.74" x2="71.12" y2="78.74" width="0.6096" layer="16"/>
-<wire x1="71.12" y1="78.74" x2="72.39" y2="77.47" width="0.6096" layer="16"/>
-<wire x1="72.39" y1="77.47" x2="72.39" y2="74.93" width="0.6096" layer="16"/>
+<wire x1="54.61" y1="77.47" x2="57.15" y2="80.01" width="0.6096" layer="16"/>
+<wire x1="57.15" y1="80.01" x2="71.12" y2="80.01" width="0.6096" layer="16"/>
+<wire x1="71.12" y1="80.01" x2="72.39" y2="78.74" width="0.6096" layer="16"/>
+<wire x1="72.39" y1="78.74" x2="72.39" y2="74.93" width="0.6096" layer="16"/>
 <wire x1="24.13" y1="77.47" x2="29.21" y2="77.47" width="0.6096" layer="16"/>
 </signal>
@@
 <wire x1="71.12" y1="72.39" x2="76.2" y2="72.39" width="0.6096" layer="16"/>
 <wire x1="76.2" y1="72.39" x2="77.47" y2="73.66" width="0.6096" layer="16"/>
-<wire x1="77.47" y1="73.66" x2="77.47" y2="81.28" width="0.6096" layer="16"/>
-<wire x1="77.47" y1="81.28" x2="76.2" y2="82.55" width="0.6096" layer="16"/>
-<wire x1="76.2" y1="82.55" x2="55.88" y2="82.55" width="0.6096" layer="16"/>
-<wire x1="55.88" y1="82.55" x2="54.61" y2="83.82" width="0.6096" layer="16"/>
-<wire x1="54.61" y1="83.82" x2="54.61" y2="87.63" width="0.6096" layer="16"/>
+<wire x1="77.47" y1="73.66" x2="77.47" y2="82.55" width="0.6096" layer="16"/>
+<wire x1="77.47" y1="82.55" x2="76.2" y2="83.82" width="0.6096" layer="16"/>
+<wire x1="76.2" y1="83.82" x2="55.88" y2="83.82" width="0.6096" layer="16"/>
+<wire x1="55.88" y1="83.82" x2="54.61" y2="85.09" width="0.6096" layer="16"/>
+<wire x1="54.61" y1="85.09" x2="54.61" y2="87.63" width="0.6096" layer="16"/>
 </signal>
 <signal name="N$26">
@@
 <wire x1="44.45" y1="74.93" x2="44.45" y2="77.47" width="0.6096" layer="16"/>
 <via x="44.45" y="77.47" extent="1-16" drill="0.6" diameter="1.6764" shape="octagon"/>
-<wire x1="44.45" y1="77.47" x2="49.53" y2="82.55" width="0.6096" layer="1"/>
-<via x="49.53" y="82.55" extent="1-16" drill="0.6" diameter="1.6764" shape="octagon"/>
-<wire x1="49.53" y1="82.55" x2="49.53" y2="87.63" width="0.6096" layer="16"/>
+<wire x1="44.45" y1="77.47" x2="49.53" y2="83.82" width="0.6096" layer="1"/>
+<via x="49.53" y="83.82" extent="1-16" drill="0.6" diameter="1.6764" shape="octagon"/>
+<wire x1="49.53" y1="83.82" x2="49.53" y2="87.63" width="0.6096" layer="16"/>
 </signal>
 <signal name="N$28">
@@
 <wire x1="30.48" y1="72.39" x2="21.59" y2="72.39" width="0.6096" layer="16"/>
 <wire x1="21.59" y1="72.39" x2="20.32" y2="73.66" width="0.6096" layer="16"/>
-<wire x1="20.32" y1="73.66" x2="20.32" y2="80.01" width="0.6096" layer="16"/>
-<wire x1="20.32" y1="80.01" x2="21.59" y2="81.28" width="0.6096" layer="16"/>
-<wire x1="21.59" y1="81.28" x2="45.72" y2="81.28" width="0.6096" layer="16"/>
-<wire x1="45.72" y1="81.28" x2="46.99" y2="82.55" width="0.6096" layer="16"/>
-<wire x1="46.99" y1="82.55" x2="46.99" y2="87.63" width="0.6096" layer="16"/>
+<wire x1="20.32" y1="73.66" x2="20.32" y2="81.28" width="0.6096" layer="16"/>
+<wire x1="20.32" y1="81.28" x2="21.59" y2="82.55" width="0.6096" layer="16"/>
+<wire x1="21.59" y1="82.55" x2="45.72" y2="82.55" width="0.6096" layer="16"/>
+<wire x1="45.72" y1="82.55" x2="46.99" y2="83.82" width="0.6096" layer="16"/>
+<wire x1="46.99" y1="83.82" x2="46.99" y2="87.63" width="0.6096" layer="16"/>
 </signal>
 <signal name="N$11">
@@
 <contactref element="IC1" pad="11"/>
 <contactref element="SV2" pad="3"/>
-<wire x1="44.45" y1="87.63" x2="44.45" y2="85.09" width="1.27" layer="16"/>
-<wire x1="44.45" y1="85.09" x2="43.18" y2="83.82" width="1.27" layer="16"/>
-<wire x1="43.18" y1="83.82" x2="15.24" y2="83.82" width="1.27" layer="16"/>
+<wire x1="44.45" y1="87.63" x2="44.45" y2="86.36" width="1.27" layer="16"/>
+<wire x1="44.45" y1="86.36" x2="43.18" y2="85.09" width="1.27" layer="16"/>
+<wire x1="43.18" y1="85.09" x2="16.51" y2="85.09" width="1.27" layer="16"/>
 <wire x1="4.5466" y1="64.135" x2="8.255" y2="64.135" width="0.6096" layer="16"/>
 <wire x1="8.255" y1="64.135" x2="8.89" y2="64.77" width="0.6096" layer="16"/>
 <wire x1="8.89" y1="64.77" x2="8.89" y2="76.835" width="0.6096" layer="16"/>
-<wire x1="19.05" y1="83.82" x2="15.24" y2="83.82" width="0.6096" layer="16"/>
 <wire x1="5.8166" y1="36.195" x2="3.175" y2="36.195" width="0.6096" layer="16"/>
 <wire x1="3.175" y1="36.195" x2="2.54" y2="36.83" width="0.6096" layer="16"/>
@@
 <via x="8.89" y="76.835" extent="1-16" drill="0.6" diameter="1.6764" shape="octagon"/>
 <wire x1="8.89" y1="76.835" x2="8.89" y2="79.375" width="0.8128" layer="16"/>
-<wire x1="8.89" y1="79.375" x2="13.335" y2="83.82" width="0.8128" layer="16"/>
-<wire x1="13.335" y1="83.82" x2="15.24" y2="83.82" width="0.8128" layer="16"/>
+<wire x1="8.89" y1="79.375" x2="14.605" y2="85.09" width="0.8128" layer="16"/>
+<wire x1="14.605" y1="85.09" x2="16.51" y2="85.09" width="0.8128" layer="16"/>
 </signal>
 <signal name="N$13">
