File: pcb/supply.sch (EAGLE design)
At the start: 28 parts, among them IC1 Lm7805, K1 ZD322006, Q6 BC548

Commit message: edit pcb
Connections:
- removed net N$16: LED1.A, R9.2
- new net N$2: LED1.C, R9.1
- net GND: now also R9.2; no longer LED1.C
- net GND1: now also R1.2; no longer LED2.C
- net N$1: now also LED2.C, R1.1; no longer LED2.A, R1.2
- net VCC: now also LED1.A, LED2.A; no longer R1.1, R9.1
Other:
- moved on the sheet: LED1, LED2, R1, R9
Changed lines of the file:
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@@
 <instance part="P+6" gate="VCC" x="165.1" y="154.94"/>
 <instance part="GND1" gate="1" x="165.1" y="106.68"/>
-<instance part="LED1" gate="G$1" x="25.4" y="142.24"/>
+<instance part="LED1" gate="G$1" x="25.4" y="157.48"/>
 <instance part="P+7" gate="VCC" x="25.4" y="165.1"/>
-<instance part="R9" gate="G$1" x="25.4" y="152.4" rot="R270"/>
+<instance part="R9" gate="G$1" x="25.4" y="144.78" rot="R270"/>
 <instance part="GND6" gate="1" x="25.4" y="132.08"/>
 <instance part="SV1" gate="G$1" x="58.42" y="45.72"/>
@@
 <instance part="X5" gate="-1" x="20.32" y="50.8"/>
 <instance part="X5" gate="-2" x="20.32" y="45.72"/>
-<instance part="LED2" gate="G$1" x="139.7" y="134.62"/>
-<instance part="R1" gate="G$1" x="139.7" y="142.24" rot="R270"/>
+<instance part="LED2" gate="G$1" x="139.7" y="144.78"/>
+<instance part="R1" gate="G$1" x="139.7" y="134.62" rot="R270"/>
 <instance part="C1" gate="G$1" x="198.12" y="134.62"/>
 <instance part="R2" gate="G$1" x="198.12" y="147.32" rot="R270"/>
@@
 </segment>
 <segment>
-<pinref part="LED1" gate="G$1" pin="C"/>
-<pinref part="GND6" gate="1" pin="GND"/>
-<wire x1="25.4" y1="137.16" x2="25.4" y2="134.62" width="0.1524" layer="91"/>
-</segment>
-<segment>
 <pinref part="GND8" gate="1" pin="GND"/>
 <wire x1="43.18" y1="33.02" x2="43.18" y2="40.64" width="0.1524" layer="91"/>
@@
 <wire x1="129.54" y1="127" x2="129.54" y2="129.54" width="0.1524" layer="91"/>
 </segment>
+<segment>
+<pinref part="GND6" gate="1" pin="GND"/>
+<pinref part="R9" gate="G$1" pin="2"/>
+<wire x1="25.4" y1="139.7" x2="25.4" y2="134.62" width="0.1524" layer="91"/>
+</segment>
 </net>
 <net name="VCC" class="0">
-<segment>
-<pinref part="R9" gate="G$1" pin="1"/>
-<pinref part="P+7" gate="VCC" pin="VCC"/>
-<wire x1="25.4" y1="157.48" x2="25.4" y2="162.56" width="0.1524" layer="91"/>
-</segment>
 <segment>
 <pinref part="P+8" gate="VCC" pin="VCC"/>
@@
 <wire x1="165.1" y1="147.32" x2="165.1" y2="152.4" width="0.1524" layer="91"/>
 <junction x="165.1" y="147.32"/>
-<pinref part="R1" gate="G$1" pin="1"/>
-<wire x1="149.86" y1="147.32" x2="139.7" y2="147.32" width="0.1524" layer="91"/>
+<pinref part="LED2" gate="G$1" pin="A"/>
+<wire x1="139.7" y1="147.32" x2="149.86" y2="147.32" width="0.1524" layer="91"/>
 <junction x="149.86" y="147.32"/>
 </segment>
@@
 <junction x="129.54" y="142.24"/>
 </segment>
-</net>
-<net name="N$16" class="0">
-<segment>
+<segment>
+<pinref part="P+7" gate="VCC" pin="VCC"/>
 <pinref part="LED1" gate="G$1" pin="A"/>
-<pinref part="R9" gate="G$1" pin="2"/>
-<wire x1="25.4" y1="144.78" x2="25.4" y2="147.32" width="0.1524" layer="91"/>
+<wire x1="25.4" y1="160.02" x2="25.4" y2="162.56" width="0.1524" layer="91"/>
 </segment>
 </net>
@@
 <net name="GND1" class="0">
 <segment>
-<pinref part="LED2" gate="G$1" pin="C"/>
-<wire x1="139.7" y1="129.54" x2="139.7" y2="127" width="0.1524" layer="91"/>
 <pinref part="Q6" gate="G$1" pin="C"/>
 <pinref part="K1" gate="1" pin="2"/>
@@
 <wire x1="149.86" y1="127" x2="139.7" y2="127" width="0.1524" layer="91"/>
 <junction x="149.86" y="127"/>
-</segment>
-</net>
-<net name="N$1" class="0">
-<segment>
-<pinref part="LED2" gate="G$1" pin="A"/>
 <pinref part="R1" gate="G$1" pin="2"/>
+<wire x1="139.7" y1="127" x2="139.7" y2="129.54" width="0.1524" layer="91"/>
 </segment>
 </net>
@@
 </segment>
 </net>
+<net name="N$1" class="0">
+<segment>
+<pinref part="LED2" gate="G$1" pin="C"/>
+<pinref part="R1" gate="G$1" pin="1"/>
+</segment>
+</net>
+<net name="N$2" class="0">
+<segment>
+<pinref part="LED1" gate="G$1" pin="C"/>
+<pinref part="R9" gate="G$1" pin="1"/>
+<wire x1="25.4" y1="149.86" x2="25.4" y2="152.4" width="0.1524" layer="91"/>
+</segment>
+</net>
